File: discipline-pcb.kicad_pcb (KiCad board)
At the start: 2 copper layers, 304.9 x 122.8 mm, 180 parts, among them J1 AVR-ISP-6, SW1 KEYSW, SW10 KEYSW, SW11 KEYSW, SW12 KEYSW, SW13 KEYSW, SW14 KEYSW, SW15 KEYSW, SW16 KEYSW, SW17 KEYSW, SW18 KEYSW, SW19 KEYSW, SW2 KEYSW, SW20 KEYSW, SW21 KEYSW, SW22 KEYSW, SW23 KEYSW, SW24 KEYSW, SW25 KEYSW, SW26 KEYSW, SW27 KEYSW, SW28 KEYSW, SW29 KEYSW, SW3 KEYSW, SW30 KEYSW, SW31 KEYSW, SW32 KEYSW, SW33 KEYSW, SW34 KEYSW, SW35 KEYSW, SW36 KEYSW, SW37 KEYSW, SW38 KEYSW, SW39 KEYSW, SW4 KEYSW, SW40 KEYSW, SW41 KEYSW, SW42 KEYSW, SW43 KEYSW, SW44 KEYSW, SW45 KEYSW, SW46 KEYSW, SW47 KEYSW, SW48 KEYSW, SW49 KEYSW, SW5 KEYSW, SW50 KEYSW, SW51 KEYSW, SW52 KEYSW, SW53 KEYSW, SW54 KEYSW, SW55 KEYSW, SW56 KEYSW, SW57 KEYSW, SW58 KEYSW, SW59 KEYSW, SW6 KEYSW, SW60 KEYSW, SW61 KEYSW, SW62 KEYSW, SW63 KEYSW, SW64 KEYSW, SW65 KEYSW, SW66 KEYSW, SW67 KEYSW, SW68 KEYSW, SW69 KEYSW, SW7 KEYSW, SW70 KEYSW, SW71 KEYSW, SW72 KEYSW, SW73 KEYSW, SW74 KEYSW, SW8 KEYSW, SW9 KEYSW, U1 ATmega32A-PU, Y1 Crystal

Commit message: Learning stuff
WIP for an attempt to create an ISO layout + split spacebar + middle
button
Parts:
- removed the G*** at (155.2, 163.6) (x2)
- removed the REF** at (184.8, 171.0)
- removed ST72: 7U, cftkb:MX-7U-Stabilizer
- removed SW70, SW74: KEYSW, cftkb:SW_Cherry_MX1A_1.50u_PCBNOSCREEN
- added D71: , cftkb:D_DO-35_SOD27_P5.08mm_Horizontal, F.Cu at (61.1, 79.1)
- added D72: , cftkb:D_DO-35_SOD27_P5.08mm_Horizontal, F.Cu at (278.6, 71.2)
- added Ref**: Val**, cftkb:credits2, F.Cu at (249.6, 158.6)
- added Ref**: Val**, cftkb:logo, F.Cu at (137.4, 158.6)
- SW29: footprint cftkb:SW_Cherry_MX1A_1.50u_PCBNOSCREEN -> cftkb:SW_Cherry_MX1A_1.25u_PCBNOSCREEN
- SW43: footprint cftkb:SW_Cherry_MX1A_2.25u_PCBNOSCREEN -> cftkb:SW_Cherry_MX1A_1.00u_PCB-NOSCREEN
- SW45: footprint cftkb:SW_Cherry_MX1A_2.25u_PCBNOSCREEN -> cftkb:SW_Cherry_MX1A_1.25u_PCBNOSCREEN
- SW59, SW60, SW61: footprint cftkb:SW_Cherry_MX1A_1.25u_PCBNOSCREEN -> cftkb:SW_Cherry_MX1A_1.00u_PCB-NOSCREEN
- SW62: footprint cftkb:SW_Cherry_MX1A_1.00u_PCB-NOSCREEN -> cftkb:SW_Cherry_MX1A_3.00u_PCB-NOSCREEN
- SW71: footprint cftkb:SW_Cherry_MX1A_1.50u_PCBNOSCREEN -> cftkb:SW_Cherry_MX1A_1.00u_PCB-NOSCREEN
- SW73: footprint cftkb:SW_Cherry_MX1A_1.50u_PCBNOSCREEN -> cftkb:SW_Cherry_MX1A_3.00u_PCB-NOSCREEN
- moved SW73 119.1 mm to (142.1, 165.9)
- moved SW62 31.0 mm to (218.3, 165.9)
- moved SW71 21.3 mm to (89.7, 146.8)
- moved SW43 11.9 mm to (308.8, 127.8)
- moved SW61 11.9 mm to (104.0, 165.9)
- moved SW29 10.9 mm to (330.2, 119.4)
- moved SW45 9.52 mm to (68.3, 146.8)
- moved SW60 7.11 mm to (85.0, 165.9)
- moved REF** 5.81 mm to (206.2, 161.1)
- moved SW59 2.37 mm to (65.9, 165.9)
- moved C4 0.05 mm to (325.1, 59.0)
Connections:
- SW43 pad 1: col13 -> col12
- SW71 pad 1: col2 -> col1
- SW71 pad 2: Net-(D61-Pad2) -> Net-(D71-Pad2)
- SW72 pad 1: col6 -> col7
- SW72 pad 2: Net-(D62-Pad2) -> Net-(D72-Pad2)
- SW73 pad 1: col9 -> col6
- SW73 pad 2: Net-(D63-Pad2) -> Net-(D62-Pad2)
Routing:
- net Net-(D72-Pad2): track 0.00 -> 335.6 mm, vias 0 -> 1
- net Net-(D71-Pad2): track 0.00 -> 79.2 mm, vias 0 -> 1
- net col6: track 279.4 -> 348.2 mm
- net col7: track 269.9 -> 308.3 mm
- net Net-(D62-Pad2): track 355.8 -> 391.4 mm
- net row4: track 296.4 -> 314.9 mm
- net row3: track 287.2 -> 301.6 mm
- net col10: track 251.0 -> 236.7 mm
- net Net-(D43-Pad2): track 140.6 -> 153.4 mm
- net Net-(D29-Pad2): track 117.7 -> 129.2 mm
- net col2: track 329.2 -> 318.0 mm
- net Net-(D63-Pad2): track 279.4 -> 268.6 mm
- net Net-(D45-Pad2): track 76.5 -> 86.2 mm
- net Net-(D59-Pad2): track 462.2 -> 454.7 mm
- net col0: track 355.0 -> 348.0 mm
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Other:
- board text removed: "1.25U"
- board text removed: "1.5U"
- board text removed: "coseyfannitutti 2019 rev1"

Commit message: Learning stuff
WIP for an attempt to create an ISO layout + split spacebar + middle
button
Parts:
- removed the Ref** at (249.6, 158.6)
- added D73: , cftkb:D_DO-35_SOD27_P5.08mm_Horizontal, F.Cu at (242.6, 79.9)
- added Ref**: Val**, cftkb:credits_mask, F.Cu at (255.7, 158.5)
- added Ref**: Val**, cftkb:credits, F.Cu at (255.7, 158.5)
- added ref_logo_mask: logo mask, cftkb:logo_mask, F.Cu at (136.4, 158.4)
- SW29: footprint cftkb:SW_Cherry_MX1A_1.25u_PCBNOSCREEN -> cftkb:SW_Cherry_MX1A_ISOEnter_PCB_ReversedStabilizer
- SW62: footprint cftkb:SW_Cherry_MX1A_3.00u_PCB-NOSCREEN -> cftkb:SW_Cherry_MX1A_1.00u_PCB-NOSCREEN
- SW72: footprint cftkb:SW_Cherry_MX1A_1.00u_PCB-NOSCREEN -> cftkb:SW_Cherry_MX1A_3.00u_PCBNOSCREEN
- SW73: footprint cftkb:SW_Cherry_MX1A_3.00u_PCB-NOSCREEN -> cftkb:SW_Cherry_MX1A_3.00u_PCBNOSCREEN
- moved D72 101.4 mm to (177.7, 80.1), turned to 180 degrees
- moved SW73 76.2 mm to (218.3, 165.9)
- moved D71 40.5 mm to (101.6, 80.1), turned to 180 degrees
- moved SW72 38.1 mm to (142.1, 165.9)
- moved SW62 38.1 mm to (180.2, 165.9)
- moved SW29 1.14 mm to (330.2, 118.2)
Connections:
- SW72 pad 1: col7 -> col5
- SW73 pad 1: col6 -> col7
- SW73 pad 2: Net-(D62-Pad2) -> Net-(D73-Pad2)
Routing:
- net Net-(D73-Pad2): track 0.00 -> 312.6 mm
- net Net-(D72-Pad2): track 335.6 -> 124.0 mm, vias 1 -> 2
- net col6: track 348.2 -> 274.6 mm
- net row4: track 314.9 -> 364.8 mm
- net col5: track 271.6 -> 306.8 mm
- net Net-(D62-Pad2): track 391.4 -> 365.8 mm, vias 0 -> 1
- net col7: track 308.3 -> 294.9 mm
- net row3: track 301.6 -> 296.7 mm
- net Net-(D68-Pad2): track 232.2 -> 234.5 mm
- net Net-(D65-Pad2): track 215.5 -> 217.2 mm
- net Net-(D66-Pad2): track 190.5 -> 192.2 mm
- net Net-(D67-Pad2): track 163.1 -> 161.7 mm
- net Net-(D58-Pad2): track 142.1 -> 140.9 mm
- net Net-(D44-Pad2): track 119.9 -> 118.7 mm
- net Net-(D61-Pad2): track 420.2 -> 419.1 mm
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Other:
- board text added: "06/07/2020"
- board text added: "The Fork of DISCIPLINE - 65% keyboard made with only through hole components Based on coseyfannitutti's DISCIPLINE Rev.1 Fork of DISCIPLINE by ikkyusan"
- board text removed: "7/2/2019"
- board text removed: "DISCIPLINE - 65% keyboard made with only through hole components"

Commit message: "Split spacebar + middle button" design completed
Re-integrated ANSI/ISO layout from coseyfannitutti v2, made some
corrections, added logo...
PCB proto is ordered, let's see how it turns out.
Parts:
- removed the Ref** at (255.7, 158.5) (x2)
- removed the Ref** at (137.4, 158.6)
- removed SW72: KEYSW, cftkb:SW_Cherry_MX1A_3.00u_PCBNOSCREEN
- removed ref_logo_mask: logo mask, cftkb:logo_mask
- added REF**: MountingHole_2.2mm_M2_Pad, cftkb:MountingHole_2.2mm_M2_Pad, F.Cu at (206.2, 80.4)
- added REF**: MountingHole_2.2mm_M2_Pad, cftkb:MountingHole_2.2mm_M2_Pad, F.Cu at (206.2, 61.7)
- added Ref**: Val**, cftkb:logo_mask, B.Cu at (132.6, 62.1)
- added Ref**: Val**, cftkb:logo, B.Cu at (132.6, 62.1)
- added Ref**: Val**, cftkb:logo, F.Cu at (265.8, 158.4)
- added Ref**: Val**, cftkb:logo_mask, F.Cu at (265.8, 158.4)
- added Ref**: Val**, cftkb:version_mask, B.Cu at (86.7, 177.2)
- added Ref**: Val**, cftkb:version, B.Cu at (86.7, 177.2)
- added SW76: KEYSW, cftkb:SW_Cherry_MX1A_ISOEnter_PCB_ReversedStabilizer, F.Cu at (330.2, 118.3)
- added SW77: KEYSW, cftkb:SW_Cherry_MX1A_1.00u_PCB-NOSCREEN, F.Cu at (308.8, 127.8)
- added SW78: KEYSW, cftkb:SW_Cherry_MX1A_1.25u_PCBNOSCREEN, F.Cu at (68.3, 146.8)
- added SW80: KEYSW, cftkb:SW_Cherry_MX1A_3.00u_PCBNOSCREEN, F.Cu at (142.1, 165.9)
- SW29: footprint cftkb:SW_Cherry_MX1A_ISOEnter_PCB_ReversedStabilizer -> cftkb:SW_Cherry_MX1A_1.50u_PCBNOSCREEN
- SW43: footprint cftkb:SW_Cherry_MX1A_1.00u_PCB-NOSCREEN -> cftkb:SW_Cherry_MX1A_2.25u_PCBNOSCREEN
- SW45: footprint cftkb:SW_Cherry_MX1A_1.25u_PCBNOSCREEN -> cftkb:SW_Cherry_MX1A_2.25u_PCBNOSCREEN
- SW63: footprint cftkb:SW_Cherry_MX1A_1.00u_PCB-NOSCREEN -> cftkb:SW_Cherry_MX1A_1.25u_PCBNOSCREEN
- moved SW43 11.9 mm to (320.7, 127.8)
- moved SW29 9.79 mm to (327.8, 108.7)
- moved SW45 9.52 mm to (77.8, 146.8)
- renumbered SW71 to SW75, SW73 to SW81
Connections:
- SW43 pad 1: col12 -> col13
Routing:
- net col13: track 140.8 -> 161.6 mm
- net col0: track 348.0 -> 355.9 mm
- net col5: track 306.8 -> 313.2 mm
- net Net-(D56-Pad2): track 142.3 -> 147.0 mm
- net Net-(D64-Pad2): track 184.8 -> 189.5 mm
- net row4: track 364.8 -> 367.0 mm
- net Net-(D57-Pad2): track 154.2 -> 152.1 mm
- net col12: track 184.7 -> 186.1 mm
- net col1: track 321.1 -> 322.4 mm
- net col2: track 318.0 -> 319.3 mm
- net col3: track 261.1 -> 262.4 mm
- net col4: track 259.3 -> 260.6 mm
- net Net-(D29-Pad2): track 129.7 -> 128.5 mm
- net Net-(D62-Pad2): track 365.8 -> 366.9 mm
- net Net-(D45-Pad2): track 86.2 -> 85.1 mm
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Other:
- board text added: "07/2020"
- board text added: "1.25U ISO"
- board text added: "1U ISO"
- board text added: "2.25U ANSI"
- board text added: "202007"
- board text added: "ANSI ENTER"
- board text added: "ISO ENTER"
- board text added: "The Fork of DISCIPLINE"
- board text added: "The Fork of DISCIPLINE - 65% keyboard made with only through hole components Based on coseyfannitutti's DISCIPLINE. https://github.com/coseyfannitutti/discipline Fork of DISCIPLINE by ikkyusan. https://github.com/ikkyusan1/discipline"
- board text removed: "06/07/2020"
- board text removed: "1"
- board text removed: "1U"
- board text removed: "The Fork of DISCIPLINE - 65% keyboard made with only through hole components Based on coseyfannitutti's DISCIPLINE Rev.1 Fork of DISCIPLINE by ikkyusan"
